Commit message: simplified environment changes.
bigger tennis balls, repositioned camera, direct cobot motor control (was end effector control before), simplified projectile motion to not hit the base.

File: cobot-env/cobot_ai4robotics/resources/projectiles/ycb_objects/YcbTennisBall/model.urdf (robot description, URDF)
Before this commit: robot model.urdf, 1 links, 0 joints
Links:
- link baseLink: geometry collision mesh filename=collision_vhacd.obj scale=5 5 5; visual mesh filename=textured_reoriented.obj scale=5 5 5

Commit message: Increased tennisball size. Added file for DQN. DQN code still in progress.

File: cobot-env/cobot_ai4robotics/resources/projectiles/ycb_objects/YcbTennisBall/model.urdf (robot description, URDF)
Before this commit: robot model.urdf, 1 links, 0 joints
Links:
- link baseLink: geometry collision mesh filename=collision_vhacd.obj scale=7 7 7; visual mesh filename=textured_reoriented.obj scale=7 7 7

Commit message: techfest

File: cobot-env/cobot_ai4robotics/resources/projectiles/ycb_objects/YcbTennisBall/model.urdf (robot description, URDF)
Before this commit: robot model.urdf, 1 links, 0 joints
Links:
- link baseLink: geometry collision mesh filename=collision_vhacd.obj scale=4 4 4; visual mesh filename=textured_reoriented.obj scale=4 4 4
